File: Power_analyzer.kicad_pcb (KiCad board)
At the start: 2 copper layers, 48.3 x 34.3 mm, 46 parts, among them J1 Conn_01x03, J2 Conn_01x03, J3 Conn_01x02, J4 Conn_01x02, J5 Conn_01x02, J6 Conn_01x03, U1 ACS712xLCTR-05B, U2 LM358, U3 ADS1115IDGS

Commit message: ????? ?????? ???????? ?? ??????????? ??????. ???????? ?????? ????? ?????????.
Parts:
- removed F1: 2A, Fuse:Fuse_Littelfuse_372_D8.50mm
- removed the J4 at (108.0, 68.1)
- removed R19, R20: 10k, Resistor_SMD:R_0603_1608Metric
- removed RV2: 10k, Potentiometer_THT:Potentiometer_Bourns_3296W_Vertical
- added C11: 100nF, Capacitor_SMD:C_0603_1608Metric, B.Cu at (111.3, 21.6)
- added J3: Conn_01x01, Connector_PinHeader_2.54mm:PinHeader_1x01_P2.54mm_Vertical, F.Cu at (84.5, 83.2)
- added U4: ADS1115IDGS, Package_SO:TSSOP-10_3x3mm_P0.5mm, F.Cu at (104.3, 20.6)
- C10, R14: moved to F.Cu
- C2: value 1nF -> 100nF
- C3: value 1uF -> 1nF; moved to F.Cu
- C5: value 1nF -> 1uF
- C6: value 1uF -> 1nF
- C7: value 1uF -> 1nF; moved to B.Cu
- C8: value 100nF -> 1uF
- C9: value 100nF -> 1uF; moved to F.Cu
- D1: footprint LED_SMD:LED_0603_1608Metric -> LED_THT:LED_D2.0mm_W4.8mm_H2.5mm_FlatTop
- J1, J2, J6: footprint Connector_PinHeader_2.54mm:PinHeader_1x03_P2.54mm_Horizontal -> Connector_PinHeader_2.54mm:PinHeader_1x03_P2.54mm_Vertical
- J4: renamed from J3; footprint Connector_PinHeader_2.54mm:PinHeader_1x02_P2.54mm_Horizontal -> Connector_PinHeader_2.54mm:PinHeader_1x02_P2.54mm_Vertical
- JP1: footprint Jumper:SolderJumper-2_P1.3mm_Open_TrianglePad1.0x1.5mm -> Jumper:SolderJumper-2_P1.3mm_Open_RoundedPad1.0x1.5mm
- R1: footprint Resistor_THT:R_Axial_DIN0516_L15.5mm_D5.0mm_P20.32mm_Horizontal -> Resistor_THT:R_Axial_DIN0516_L15.5mm_D5.0mm_P5.08mm_Vertical
- R6: value 100k -> 10k; moved to B.Cu
- R7: value 10k -> 100k; moved to F.Cu
- RV1: value Varistor -> 10k; footprint Varistor:RV_Disc_D12mm_W5.1mm_P7.5mm -> Potentiometer_THT:Potentiometer_Bourns_3296W_Vertical
- U2: value LM358 -> ACS712xLCTR-05B
- U3: value ADS1115IDGS -> LM358; footprint Package_SO:TSSOP-10_3x3mm_P0.5mm -> Package_SO:SOIC-8_3.9x4.9mm_P1.27mm
- moved R12 67.2 mm to (52.8, 28.1)
- moved R18 63.8 mm to (52.8, 28.1)
- moved C8 61.5 mm to (52.8, 28.1), turned to 0 degrees
- moved RV1 59.7 mm to (52.8, 28.1), turned to 90 degrees
- moved C6 59.3 mm to (52.8, 28.1), turned to 270 degrees
- moved R15 59.2 mm to (52.8, 28.1), turned to 90 degrees
- moved C2 58.5 mm to (52.8, 28.1)
- moved C9 58.2 mm to (52.8, 28.1), turned to 270 degrees
- moved R14 57.4 mm to (52.8, 28.1), turned to 180 degrees
- moved R10 56.8 mm to (52.8, 28.1)
- moved J5 55.9 mm to (52.8, 28.1)
- moved C3 54.8 mm to (132.5, 40.2)
- moved R17 52.5 mm to (89.3, 18.6), turned to 270 degrees
- moved R5 49.1 mm to (52.8, 28.1)
- moved C10 47.7 mm to (66.3, 29.6), turned to 90 degrees
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Connections:
- C10 pad 1: GND -> +5VP
- C10 pad 2: +5VP -> Net-(C10-Pad2)
- C2 pad 1: Net-(C2-Pad1) -> +5VP
- C3 pad 2: Net-(C3-Pad2) -> GND
- C4 pad 2: Net-(C4-Pad2) -> GND
- C5 pad 1: GND -> Net-(C5-Pad1)
- C5 pad 2: +5VP -> Net-(C5-Pad2)
- C7 pad 1: /Uin -> GND
- C7 pad 2: Net-(C6-Pad1) -> +5VP
- C8 pad 1: +5VP -> Net-(C8-Pad1)
- C9 pad 1: +5VP -> /UL1
- C9 pad 2: Net-(C9-Pad2) -> Net-(C8-Pad1)
- J1 pad 1: /N -> Net-(J1-Pad1)
- J1 pad 2: Net-(J1-Pad2) -> /L1
- J1 pad 3: Net-(F1-Pad1) -> (no net)
- J2 pad 1: /N -> Net-(J2-Pad1)
- J2 pad 3: /L -> (no net)
- J5 pad 1: Net-(C9-Pad2) -> Net-(C10-Pad2)
- PT1 pad 2: /N -> Net-(J3-Pad1)
- PT1 pad 4: Net-(C3-Pad1) -> Net-(C5-Pad1)
- R1 pad 2: /L -> /L1
- R10 pad 1: /Uin -> /UL1
- R10 pad 2: Net-(C6-Pad1) -> Net-(C8-Pad1)
- R11 pad 1: /Uin -> /UL1
- R12 pad 2: Net-(C8-Pad2) -> Net-(C10-Pad2)
- R13 pad 1: Net-(C8-Pad2) -> Net-(C10-Pad2)
- R14 pad 1: +5VP -> GND
- R14 pad 2: Net-(C9-Pad2) -> Net-(JP2-Pad1)
- R15 pad 1: Net-(C9-Pad2) -> +5VP
- R15 pad 2: GND -> Net-(J6-Pad1)
- R16 pad 1: GND -> +5VP
- R16 pad 2: Net-(JP2-Pad1) -> Net-(J6-Pad2)
- R17 pad 1: +5VP -> Net-(JP2-Pad3)
- R17 pad 2: Net-(J6-Pad1) -> +5VP
- R18 pad 2: Net-(J6-Pad2) -> Net-(J6-Pad3)
- R2 pad 2: Net-(C3-Pad1) -> Net-(C5-Pad1)
- R3 pad 1: Net-(C4-Pad2) -> Net-(C6-Pad2)
- R3 pad 2: Net-(C3-Pad2) -> Net-(C5-Pad2)
- R6 pad 1: Net-(C4-Pad1) -> Net-(D1-Pad2)
- R6 pad 2: Net-(C4-Pad2) -> Net-(JP1-Pad2)
- R7 pad 1: Net-(D1-Pad2) -> Net-(C6-Pad1)
- R7 pad 2: Net-(JP1-Pad2) -> Net-(C6-Pad2)
- RV1 pad 1: Net-(F1-Pad2) -> Net-(C6-Pad1)
- RV1 pad 2: /N -> Net-(C8-Pad2)
- U1 pad 1: Net-(F1-Pad2) -> Net-(J1-Pad1)
- U1 pad 2: Net-(F1-Pad2) -> Net-(J1-Pad1)
- U1 pad 3: /L -> /L1
- U1 pad 4: /L -> /L1
- U1 pad 6: Net-(C2-Pad1) -> Net-(C3-Pad1)
- U1 pad 7: /Iin -> /I_L1
- U2 pad 1: Net-(C4-Pad1) -> Net-(J2-Pad1)
- U2 pad 2: Net-(C4-Pad2) -> Net-(J2-Pad1)
- U2 pad 3: Net-(R4-Pad1) -> Net-(J2-Pad2)
- U2 pad 4: GND -> Net-(J2-Pad2)
- U2 pad 5: Net-(R8-Pad1) -> GND
- U2 pad 6: Net-(C6-Pad1) -> Net-(C4-Pad1)
- U2 pad 7: /Uin -> (no net)
- U3 pad 1: Net-(JP2-Pad2) -> Net-(C6-Pad1)
- U3 pad 2: Net-(J6-Pad1) -> Net-(C6-Pad2)
- U3 pad 3: GND -> Net-(R4-Pad1)
- U3 pad 4: /Uin -> GND
- U3 pad 5: /Iin -> Net-(R8-Pad1)
- U3 pad 6: Net-(C9-Pad2) -> Net-(C8-Pad1)
- U3 pad 7: Net-(C8-Pad2) -> /UL1
Routing:
- net GND: track 67.6 -> 0.00 mm, vias 3 -> 0
- net +5VP: track 48.6 -> 0.00 mm, vias 4 -> 0
- net Net-(J6-Pad1): track 23.2 -> 0.00 mm, vias 1 -> 0
- net Net-(C4-Pad1): track 21.0 -> 0.00 mm, vias 1 -> 0
- net Net-(C8-Pad2): track 18.7 -> 0.00 mm, vias 1 -> 0
- net Net-(J6-Pad2): track 17.7 -> 0.00 mm, vias 1 -> 0
- net Net-(J6-Pad3): track 17.6 -> 0.00 mm, vias 1 -> 0
- net /Uin: track 14.7 -> 0.00 mm, vias 1 -> 0
- net /Iin: track 14.3 -> 0.00 mm, vias 2 -> 0
- net Net-(C9-Pad2): track 12.9 -> 0.00 mm
- net Net-(C4-Pad2): track 11.4 -> 0.00 mm, vias 1 -> 0
- net Net-(R4-Pad1): track 11.3 -> 0.00 mm, vias 1 -> 0
- net Net-(C6-Pad1): track 6.34 -> 0.00 mm
- net Net-(R8-Pad1): track 5.13 -> 0.00 mm, vias 1 -> 0
- net Net-(C6-Pad2): track 3.93 -> 0.00 mm
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- removed copper zone on B.Cu, net +5VP
- removed copper zone on F.Cu, net /L
- removed copper zone on B.Cu, net /N
- removed copper zone on F.Cu, net GND
- removed copper zone on B.Cu, net Net-(C3-Pad1)
- removed copper zone on F.Cu, net Net-(F1-Pad1)
- removed copper zone on B.Cu, net Net-(F1-Pad2)
- removed copper zone on F.Cu, net Net-(F1-Pad2)
- removed copper zone on F.Cu, net Net-(PT1-Pad1)
- removed copper zone on B.Cu, net Net-(PT1-Pad3)
Other:
- board size 48.3 x 34.3 mm -> 48.3 x 25.4 mm

Commit message: ????????????? ????? ??????????? ???????? ??????????.
Parts:
- removed the R6 at (74.0, 41.2)
- added J7: Conn_01x03, Modules:PinHeader_1x03_P2.54mm, F.Cu at (100.3, 83.2)
- added J8: Conn_01x02, Connector_JST:JST_EH_B2B-EH-A_1x02_P2.50mm_Vertical, F.Cu at (97.3, 65.5)
- added R7: 10k, Resistor_SMD:R_0603_1608Metric, B.Cu at (77.5, 61.3)
- C1, C10, C2, C3, C4, C6, C8, C9, R10, R12, R16, R17, R18, R5, U1, U2, U3, U4: moved to B.Cu
- D1, JP1, R9: moved to F.Cu
- J1, J2: value Conn_01x03 -> Conn_01x01; footprint Connector_PinHeader_2.54mm:PinHeader_1x03_P2.54mm_Vertical -> Modules:PinHeader_1x01_P2.54mm
- J3: footprint Connector_PinHeader_2.54mm:PinHeader_1x01_P2.54mm_Vertical -> Modules:PinHeader_1x01_P2.54mm
- J4: value Conn_01x02 -> Conn_01x01; footprint Connector_PinHeader_2.54mm:PinHeader_1x02_P2.54mm_Vertical -> Modules:PinHeader_1x01_P2.54mm
- J5: value Conn_01x02 -> Conn_01x01; footprint Connector_JST:JST_EH_B2B-EH-A_1x02_P2.50mm_Vertical -> Modules:PinHeader_1x01_P2.54mm
- J6: value Conn_01x03 -> Conn_01x02; footprint Connector_PinHeader_2.54mm:PinHeader_1x03_P2.54mm_Vertical -> Modules:PinHeader_1x02_P2.54mm
- R1: footprint Resistor_THT:R_Axial_DIN0516_L15.5mm_D5.0mm_P5.08mm_Vertical -> Resistor_THT:R_Axial_DIN0309_L9.0mm_D3.2mm_P5.08mm_Vertical
- R6: renamed from R7; moved to B.Cu
- moved C3 72.9 mm to (66.0, 70.2), turned to 90 degrees
- moved R15 66.8 mm to (101.6, 73.8), turned to 270 degrees
- moved R14 65.5 mm to (97.3, 76.1), turned to 270 degrees
- moved R18 61.9 mm to (100.8, 67.2), turned to 270 degrees
- moved C8 60.6 mm to (99.3, 66.9), turned to 90 degrees
- moved C9 60.3 mm to (97.5, 68.5), turned to 90 degrees
- moved R17 59.1 mm to (94.9, 77.3), turned to 180 degrees
- moved R10 59.0 mm to (95.8, 68.5), turned to 90 degrees
- moved J5 58.1 mm to (71.1, 83.2), turned to 0 degrees
- moved C2 57.4 mm to (88.9, 72.8), turned to 90 degrees
- moved R9 55.4 mm to (97.5, 72.8), turned to 90 degrees
- moved JP2 55.1 mm to (97.2, 80.6)
- moved C4 54.3 mm to (81.8, 74.0), turned to 90 degrees
- moved R2 53.5 mm to (79.3, 71.0)
- moved C6 53.3 mm to (86.4, 69.5), turned to 90 degrees
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Connections:
- C10 pad 2: Net-(C10-Pad2) -> /U_th
- C9 pad 1: /UL1 -> /U_L1
- J1 pad 1: Net-(J1-Pad1) -> /L1
- J2 pad 1: Net-(J2-Pad1) -> /L1in
- J3 pad 1: Net-(J3-Pad1) -> /L2
- J4 pad 1: GND -> /L2in
- J5 pad 1: Net-(C10-Pad2) -> /N1
- J6 pad 1: Net-(J6-Pad1) -> +5VP
- J6 pad 2: Net-(J6-Pad2) -> GND
- PT1 pad 2: Net-(J3-Pad1) -> /N1
- R10 pad 1: /UL1 -> /U_L1
- R11 pad 1: /UL1 -> /U_L1
- R12 pad 2: Net-(C10-Pad2) -> /U_th
- R13 pad 1: Net-(C10-Pad2) -> /U_th
- R15 pad 2: Net-(J6-Pad1) -> /~RDY
- R16 pad 2: Net-(J6-Pad2) -> /SCL
- R18 pad 2: Net-(J6-Pad3) -> /SDA
- U1 pad 1: Net-(J1-Pad1) -> /L1
- U1 pad 2: Net-(J1-Pad1) -> /L1
- U1 pad 3: /L1 -> /L1in
- U1 pad 4: /L1 -> /L1in
- U2 pad 1: Net-(J2-Pad1) -> /L2
- U2 pad 2: Net-(J2-Pad1) -> /L2
- U2 pad 3: Net-(J2-Pad2) -> /L2in
- U2 pad 4: Net-(J2-Pad2) -> /L2in
- U2 pad 7: (no net) -> /I_L2
- U3 pad 7: /UL1 -> /U_L1
- U4 pad 10: Net-(J6-Pad2) -> /SCL
- U4 pad 2: Net-(J6-Pad1) -> /~RDY
- U4 pad 5: (no net) -> /I_L2
- U4 pad 6: (no net) -> /U_L1
- U4 pad 7: Net-(C10-Pad2) -> /U_th
- U4 pad 9: Net-(J6-Pad3) -> /SDA
Routing:
- net GND: track 0.00 -> 96.6 mm, vias 0 -> 4
- net +5VP: track 0.00 -> 91.5 mm, vias 0 -> 8
- net /I_L1: track 0.00 -> 55.5 mm, vias 0 -> 4
- net /U_th: track 0.00 -> 30.2 mm, vias 0 -> 2
- net /SCL: track 0.00 -> 23.1 mm
- net /L1: track 0.00 -> 20.8 mm
- net /SDA: track 0.00 -> 17.5 mm, vias 0 -> 1
- net /I_L2: track 0.00 -> 16.6 mm, vias 0 -> 2
- net Net-(C8-Pad2): track 0.00 -> 13.7 mm
- net Net-(C6-Pad1): track 0.00 -> 13.5 mm
- net /U_L1: track 0.00 -> 12.6 mm
- net Net-(R4-Pad1): track 0.00 -> 10.4 mm
- net Net-(PT1-Pad3): track 0.00 -> 10.1 mm
- net Net-(R8-Pad1): track 0.00 -> 9.91 mm, vias 0 -> 2
- net /~RDY: track 0.00 -> 9.11 mm
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- added copper zone on B.Cu, net /L1
- added copper zone on B.Cu, net /L1in
- added copper zone on B.Cu, net /L2
- added copper zone on B.Cu, net /L2in
- added copper zone on B.Cu, net /N1
Other:
- board text added: "L1in"
- board text added: "L1out"
- board text added: "L2in"
- board text added: "L2out"
- board text removed: "L"
