File: Power_analyzer.sch (KiCad schematic (older format))
At the start: 46 parts, among them J1 Conn_01x03, J2 Conn_01x03, J3 Conn_01x02, J4 Conn_01x02, J5 Conn_01x02, J6 Conn_01x03, U1 ACS712xLCTR-05B, U2 LM358, U3 ADS1115IDGS

Commit message: ????? ?????? ???????? ?? ??????????? ??????. ???????? ?????? ????? ?????????.
Parts:
- removed C9: 100nF, Capacitor_SMD:C_0603_1608Metric, symbol Device:C_Small
- removed F1: 2A, Fuse:Fuse_Littelfuse_372_D8.50mm, symbol Device:Fuse_Small
- removed J5: Conn_01x02, Connector_JST:JST_EH_B2B-EH-A_1x02_P2.50mm_Vertical, symbol Connector_Generic:Conn_01x02
- removed R14, R15: 10k, Resistor_SMD:R_0603_1608Metric, symbol Device:R_Small
- removed RV1: Varistor, Varistor:RV_Disc_D12mm_W5.1mm_P7.5mm, symbol Device:Varistor
- added C2: 100nF, Capacitor_SMD:C_0603_1608Metric, symbol Device:C_Small
- added C4: 1nF, Capacitor_SMD:C_0603_1608Metric, symbol Device:C_Small
- added J3: Conn_01x01, Connector_PinHeader_2.54mm:PinHeader_1x01_P2.54mm_Vertical, symbol Connector_Generic:Conn_01x01
- added U2: ACS712xLCTR-05B, Package_SO:SOIC-8_3.9x4.9mm_P1.27mm, symbol Sensor_Current:ACS712xLCTR-05B
- J1, J2, J6: footprint Connector_PinHeader_2.54mm:PinHeader_1x03_P2.54mm_Horizontal -> Connector_PinHeader_2.54mm:PinHeader_1x03_P2.54mm_Vertical
- J4: renamed from J3; footprint Connector_PinHeader_2.54mm:PinHeader_1x02_P2.54mm_Horizontal -> Connector_PinHeader_2.54mm:PinHeader_1x02_P2.54mm_Vertical
- renumbered C8 to C10, C10 to C11, C2 to C3, C3 to C5, C4 to C6, C5 to C7, C6 to C8, C7 to C9, J4 to J5, R16 to R14, R17 to R15, R18 to R16, R19 to R17, R20 to R18, R7 to R6, R6 to R7, RV2 to RV1, U2 to U3, U3 to U4
Connections:
- net +5VP: now also C2.1, U2.8 (VCC)
- net GND: now also C2.2, C4.2, U2.5 (GND)
- net at U1.1 (IP+), U1.2 (IP+): now also J1.1 (Pin_1)
- net L1: now reaches J1.2 (Pin_2)
- net L1: now also R1.2, U1.3 (IP-), U1.4 (IP-)
- net at J2.2 (Pin_2): now also U2.3 (IP-), U2.4 (IP-)
- net U_L1: now reaches U4.6 (AIN2)
- net Iin renamed I_L1
- net I_L1: now also U4.4 (AIN0); no longer U4.5 (AIN1)
- removed net L: J2.3 (Pin_3), R1.2, U1.3 (IP-), U1.4 (IP-)
- removed net N: J1.1 (Pin_1), J2.1 (Pin_1), PT1.2
- net Uin renamed UL1
- net UL1: no longer U4.4 (AIN0)
- new net: J3.1 (Pin_1), PT1.2
- new net: J2.1 (Pin_1), U2.1 (IP+), U2.2 (IP+)
- new net: C4.1, U2.6 (FILTER)
- new net IL2: U2.7 (VIOUT)
- new net I_L2: U4.5 (AIN1)
Other:
- moved on the sheet: C10, C11, D1, J1, J5, J6, JP1, JP2, R12, R13, R14, R15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

Commit message: ????????????? ????? ??????????? ???????? ??????????.
Parts:
- removed J1, J2, J6: Conn_01x03, Connector_PinHeader_2.54mm:PinHeader_1x03_P2.54mm_Vertical, symbol Connector_Generic:Conn_01x03
- removed J4: Conn_01x02, Connector_PinHeader_2.54mm:PinHeader_1x02_P2.54mm_Vertical, symbol Connector_Generic:Conn_01x02
- added J1, J2, J4, J5: Conn_01x01, Modules:PinHeader_1x01_P2.54mm, symbol Connector_Generic:Conn_01x01
- added J6: Conn_01x02, Modules:PinHeader_1x02_P2.54mm, symbol Connector_Generic:Conn_01x02
- added J7: Conn_01x03, Modules:PinHeader_1x03_P2.54mm, symbol Connector_Generic:Conn_01x03
- J3: footprint Connector_PinHeader_2.54mm:PinHeader_1x01_P2.54mm_Vertical -> Modules:PinHeader_1x01_P2.54mm
- R1: footprint Resistor_THT:R_Axial_DIN0516_L15.5mm_D5.0mm_P20.32mm_Horizontal -> Resistor_THT:R_Axial_DIN0309_L9.0mm_D3.2mm_P5.08mm_Vertical
- renumbered J5 to J8, R7 to R6, R6 to R7
Connections:
- net IL2 is gone; now on net I_L2: U2.7 (VIOUT)
- net UL1 is gone; now on net U_L1: C9.1, R10.1, R11.1, U3.7
- net +5VP: now also J6.1 (Pin_1)
- net GND: now also J6.2 (Pin_2)
- net L1: now also U1.1 (IP+), U1.2 (IP+), J1.1 (Pin_1); no longer U1.3 (IP-), U1.4 (IP-)
- net L2: now reaches J3.1 (Pin_1)
- net L2: now also U2.1 (IP+), U2.2 (IP+); no longer PT1.2
- net L2in: now reaches U2.3 (IP-), U2.4 (IP-)
- net L2in: now also J4.1 (Pin_1)
- net SCL: now reaches R16.2, U4.10 (SCL)
- net SCL: now also J7.1 (Pin_1)
- net ~RDY: now reaches R15.2, U4.2 (ALERT/RDY)
- net ~RDY: now also J7.3 (Pin_3)
- net U_th: now reaches C10.2, J8.1 (Pin_1), R12.2, R13.1, U4.7 (AIN3)
- net SDA: now reaches R18.2, U4.9 (SDA)
- net SDA: now also J7.2 (Pin_2)
- new net L1in: J2.1 (Pin_1), U1.3 (IP-), U1.4 (IP-)
- new net N1: J5.1 (Pin_1), PT1.2
- no-connect marks 2 -> 0
Other:
- moved on the sheet: C1, C10, C11, C2, C3, C4, C5, C6, C7, C8, C9, D1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
